Commit message: Update

File: 106.URDF (robot description, URDF)
Before this commit: robot 106, 17 links, 0 joints
Links:
- removed link 10_caster
- removed link 11_base
- removed link 12_gas lift piece
- removed link 13_gas lift piece
- removed link 14_arm
- removed link 15_arm
- removed link 16_back
- removed link 17_seat
- removed link 1_wheel
- removed link 2_caster
- removed link 3_wheel
- removed link 4_caster
- removed link 5_wheel
- removed link 6_caster
- removed link 7_wheel
- removed link 8_caster
- removed link 9_wheel
- added link arm14; visual mesh filename=./raw_data/part_dae/14.dae
- added link arm15; visual mesh filename=./raw_data/part_dae/15.dae
- added link back16; visual mesh filename=./raw_data/part_dae/16.dae
- added link base11; visual mesh filename=./raw_data/part_dae/11.dae
- added link caster10; visual mesh filename=./raw_data/part_dae/10.dae
- added link caster2; visual mesh filename=./raw_data/part_dae/2.dae
- added link caster4; visual mesh filename=./raw_data/part_dae/4.dae
- added link caster6; visual mesh filename=./raw_data/part_dae/6.dae
- added link caster8; visual mesh filename=./raw_data/part_dae/8.dae
- added link gas lift piece12; visual mesh filename=./raw_data/part_dae/12.dae
- added link gas lift piece13; visual mesh filename=./raw_data/part_dae/13.dae
- added link seat17; visual mesh filename=./raw_data/part_dae/17.dae
- added link wheel1; visual mesh filename=./raw_data/part_dae/1.dae
- added link wheel3; visual mesh filename=./raw_data/part_dae/3.dae
- added link wheel5; visual mesh filename=./raw_data/part_dae/5.dae
- added link wheel7; visual mesh filename=./raw_data/part_dae/7.dae
- added link wheel9; visual mesh filename=./raw_data/part_dae/9.dae
Joints:
- added joint arm14_back16: type fixed, parent arm14, child back16, origin xyz=0.0 0.0 0.0 rpy=0 0 0
- added joint arm15_back16: type fixed, parent arm15, child back16, origin xyz=0.0 0.0 0.0 rpy=0 0 0
- added joint base11_wheel5: type fixed, parent base11, child wheel5, origin xyz=-0.26165415346622467 -1.8829651171614614e-09 -0.086154505610466 rpy=0 0 0
- added joint caster10_base11: type fixed, parent caster10, child base11, origin xyz=0.0 0.0 0.0 rpy=0 0 0
- added joint caster10_wheel9_rotation: type revolute, parent caster10, child wheel9, origin xyz=0.00319099985063076 -9.658934985168344e-09 -0.441940002143383 rpy=0 0 0, axis 1.0 0.0 0.0, limit lower=-3.141592653589793 upper=3.141592653589793 effort=10 velocity=3
- added joint caster2_base11: type fixed, parent caster2, child base11, origin xyz=0.0 0.0 0.0 rpy=0 0 0
- added joint caster2_wheel1_rotation: type revolute, parent caster2, child wheel1, origin xyz=0.16592684388160706 -4.846891027421307e-09 -0.22176782367751002 rpy=0 0 0, axis 1.0 0.0 0.0, limit lower=-3.141592653589793 upper=3.141592653589793 effort=10 velocity=3
- added joint caster4_base11: type fixed, parent caster4, child base11, origin xyz=0.0 0.0 0.0 rpy=0 0 0
- added joint caster4_wheel3_rotation: type revolute, parent caster4, child wheel3, origin xyz=0.06868565082550049 -0.39346974258781975 0.2537205144762993 rpy=0 0 0, axis 1.0 0.0 0.0, limit lower=-3.141592653589793 upper=3.141592653589793 effort=10 velocity=3
- added joint caster6_base11: type fixed, parent caster6, child base11, origin xyz=0.0 0.0 0.0 rpy=0 0 0
- added joint caster6_wheel5_rotation: type revolute, parent caster6, child wheel5, origin xyz=-0.26165415346622467 -1.8829651171614614e-09 -0.086154505610466 rpy=0 0 0, axis 1.0 0.0 0.0, limit lower=-3.141592653589793 upper=3.141592653589793 effort=10 velocity=3
- added joint caster8_base11: type fixed, parent caster8, child base11, origin xyz=0.0 0.0 0.0 rpy=0 0 0
- added joint caster8_wheel7_rotation: type revolute, parent caster8, child wheel7, origin xyz=-0.26165415346622467 -7.880555097372621e-09 -0.3605721518397331 rpy=0 0 0, axis 1.0 0.0 0.0, limit lower=-3.141592653589793 upper=3.141592653589793 effort=10 velocity=3
- added joint gas lift piece12_base11: type fixed, parent gas lift piece12, child base11, origin xyz=0.0 0.0 0.0 rpy=0 0 0
- added joint gas lift piece12_gas lift piece13_prismatic: type prismatic, parent gas lift piece12, child gas lift piece13, origin xyz=-0.06868569145071565 0.26775474017025536 -0.22430335969031795 rpy=0 0 0, axis 0.0 1.0 0.0, limit lower=-0.0365284856855869 upper=0.00347151431441307 effort=10 velocity=3
- added joint gas lift piece13_seat17_rotation: type revolute, parent gas lift piece13, child seat17, origin xyz=0.0 0.4177574962377548 -0.002097010612487793 rpy=0 0 0, axis 0.0 1.0 0.0, limit lower=-3.141592653589793 upper=3.141592653589793 effort=10 velocity=3
- added joint seat17_arm14: type fixed, parent seat17, child arm14, origin xyz=0.0 0.0 0.0 rpy=0 0 0
- added joint seat17_arm15: type fixed, parent seat17, child arm15, origin xyz=0.0 0.0 0.0 rpy=0 0 0
- added joint seat17_back16: type fixed, parent seat17, child back16, origin xyz=0.0 0.0 0.0 rpy=0 0 0

Commit message: Fix bug

File: 106.URDF (robot description, URDF)
Before this commit: robot 106, 17 links, 19 joints
Joints:
- joint gas lift piece13_seat17_rotation: origin xyz=0.0 0.4177574962377548 -0.002097010612487793 rpy=0 0 0 -> xyz=0.06868569145071565 0.15000275606749947 0.22220634907783016 rpy=0 0 0
- joint seat17_arm14: origin xyz=0.0 0.0 0.0 rpy=0 0 0 -> xyz=0.0 -0.4177574962377548 0.002097010612487793 rpy=0 0 0
- joint seat17_arm15: origin xyz=0.0 0.0 0.0 rpy=0 0 0 -> xyz=0.0 -0.4177574962377548 0.002097010612487793 rpy=0 0 0
- joint seat17_back16: origin xyz=0.0 0.0 0.0 rpy=0 0 0 -> xyz=0.0 -0.4177574962377548 0.002097010612487793 rpy=0 0 0

Commit message: update dae

File: 106.URDF (robot description, URDF)
Before this commit: robot 106, 17 links, 19 joints
Links:
- removed link arm14
- removed link arm15
- removed link back16
- removed link base11
- removed link caster10
- removed link caster2
- removed link caster4
- removed link caster6
- removed link gas lift piece12
- removed link gas lift piece13
- removed link seat17
- removed link wheel1
- removed link wheel3
- removed link wheel5
- removed link wheel9
Joints:
- removed joint arm14_back16
- removed joint arm15_back16
- removed joint base11_wheel5
- removed joint caster10_base11
- removed joint caster10_wheel9_rotation
- removed joint caster2_base11
- removed joint caster2_wheel1_rotation
- removed joint caster4_base11
- removed joint caster4_wheel3_rotation
- removed joint caster6_base11
- removed joint caster6_wheel5_rotation
- removed joint caster8_base11
- removed joint gas lift piece12_base11
- removed joint gas lift piece12_gas lift piece13_prismatic
- removed joint gas lift piece13_seat17_rotation
- removed joint seat17_arm14
- removed joint seat17_arm15
- removed joint seat17_back16

Commit message: delete not useful file

File: 106.URDF (robot description, URDF)
Before this commit: robot 106, 2 links, 1 joints
Links:
- added link arm14; visual mesh filename=./raw_data/part_dae/14.dae
- added link arm15; visual mesh filename=./raw_data/part_dae/15.dae
- added link back16; visual mesh filename=./raw_data/part_dae/16.dae
- added link base11; visual mesh filename=./raw_data/part_dae/11.dae
- added link caster10; visual mesh filename=./raw_data/part_dae/10.dae
- added link caster2; visual mesh filename=./raw_data/part_dae/2.dae
- added link caster4; visual mesh filename=./raw_data/part_dae/4.dae
- added link caster6; visual mesh filename=./raw_data/part_dae/6.dae
- added link gas lift piece12; visual mesh filename=./raw_data/part_dae/12.dae
- added link gas lift piece13; visual mesh filename=./raw_data/part_dae/13.dae
- added link seat17; visual mesh filename=./raw_data/part_dae/17.dae
- added link wheel1; visual mesh filename=./raw_data/part_dae/1.dae
- added link wheel3; visual mesh filename=./raw_data/part_dae/3.dae
- added link wheel5; visual mesh filename=./raw_data/part_dae/5.dae
- added link wheel9; visual mesh filename=./raw_data/part_dae/9.dae
Joints:
- added joint arm14_back16: type fixed, parent arm14, child back16, origin xyz=0.0 0.0 0.0 rpy=0 0 0
- added joint arm15_back16: type fixed, parent arm15, child back16, origin xyz=0.0 0.0 0.0 rpy=0 0 0
- added joint base11_wheel5: type fixed, parent base11, child wheel5, origin xyz=-0.26165415346622467 -1.8829651171614614e-09 -0.086154505610466 rpy=0 0 0
- added joint caster10_base11: type fixed, parent caster10, child base11, origin xyz=0.0 0.0 0.0 rpy=0 0 0
- added joint caster10_wheel9_rotation: type revolute, parent caster10, child wheel9, origin xyz=0.00319099985063076 -9.658934985168344e-09 -0.441940002143383 rpy=0 0 0, axis 1.0 0.0 0.0, limit lower=-3.141592653589793 upper=3.141592653589793 effort=10 velocity=3
- added joint caster2_base11: type fixed, parent caster2, child base11, origin xyz=0.0 0.0 0.0 rpy=0 0 0
- added joint caster2_wheel1_rotation: type revolute, parent caster2, child wheel1, origin xyz=0.16592684388160706 -4.846891027421307e-09 -0.22176782367751002 rpy=0 0 0, axis 1.0 0.0 0.0, limit lower=-3.141592653589793 upper=3.141592653589793 effort=10 velocity=3
- added joint caster4_base11: type fixed, parent caster4, child base11, origin xyz=0.0 0.0 0.0 rpy=0 0 0
- added joint caster4_wheel3_rotation: type revolute, parent caster4, child wheel3, origin xyz=0.06868565082550049 -0.39346974258781975 0.2537205144762993 rpy=0 0 0, axis 1.0 0.0 0.0, limit lower=-3.141592653589793 upper=3.141592653589793 effort=10 velocity=3
- added joint caster6_base11: type fixed, parent caster6, child base11, origin xyz=0.0 0.0 0.0 rpy=0 0 0
- added joint caster6_wheel5_rotation: type revolute, parent caster6, child wheel5, origin xyz=-0.26165415346622467 -1.8829651171614614e-09 -0.086154505610466 rpy=0 0 0, axis 1.0 0.0 0.0, limit lower=-3.141592653589793 upper=3.141592653589793 effort=10 velocity=3
- added joint caster8_base11: type fixed, parent caster8, child base11, origin xyz=0.0 0.0 0.0 rpy=0 0 0
- added joint gas lift piece12_base11: type fixed, parent gas lift piece12, child base11, origin xyz=0.0 0.0 0.0 rpy=0 0 0
- added joint gas lift piece12_gas lift piece13_prismatic: type prismatic, parent gas lift piece12, child gas lift piece13, origin xyz=-0.06868569145071565 0.26775474017025536 -0.22430335969031795 rpy=0 0 0, axis 0.0 1.0 0.0, limit lower=-0.0365284856855869 upper=0.00347151431441307 effort=10 velocity=3
- added joint gas lift piece13_seat17_rotation: type revolute, parent gas lift piece13, child seat17, origin xyz=0.06868569145071565 0.15000275606749947 0.22220634907783016 rpy=0 0 0, axis 0.0 1.0 0.0, limit lower=-3.141592653589793 upper=3.141592653589793 effort=10 velocity=3
- added joint seat17_arm14: type fixed, parent seat17, child arm14, origin xyz=0.0 -0.4177574962377548 0.002097010612487793 rpy=0 0 0
- added joint seat17_arm15: type fixed, parent seat17, child arm15, origin xyz=0.0 -0.4177574962377548 0.002097010612487793 rpy=0 0 0
- added joint seat17_back16: type fixed, parent seat17, child back16, origin xyz=0.0 -0.4177574962377548 0.002097010612487793 rpy=0 0 0

Commit message: update the name of the link and joint

File: 106.URDF (robot description, URDF)
Before this commit: robot 106, 17 links, 19 joints
Links:
- removed link arm14
- removed link arm15
- removed link back16
- removed link base11
- removed link caster10
- removed link caster2
- removed link caster4
- removed link caster6
- removed link caster8
- removed link gas lift piece12
- removed link gas lift piece13
- removed link seat17
- removed link wheel1
- removed link wheel3
- removed link wheel5
- removed link wheel7
- removed link wheel9
- added link 10:caster; visual mesh filename=./raw_data/part_dae/10.dae
- added link 11:base; visual mesh filename=./raw_data/part_dae/11.dae
- added link 12:gas lift piece; visual mesh filename=./raw_data/part_dae/12.dae
- added link 13:gas lift piece; visual mesh filename=./raw_data/part_dae/13.dae
- added link 14:arm; visual mesh filename=./raw_data/part_dae/14.dae
- added link 15:arm; visual mesh filename=./raw_data/part_dae/15.dae
- added link 16:back; visual mesh filename=./raw_data/part_dae/16.dae
- added link 17:seat; visual mesh filename=./raw_data/part_dae/17.dae
- added link 1:wheel; visual mesh filename=./raw_data/part_dae/1.dae
- added link 2:caster; visual mesh filename=./raw_data/part_dae/2.dae
- added link 3:wheel; visual mesh filename=./raw_data/part_dae/3.dae
- added link 4:caster; visual mesh filename=./raw_data/part_dae/4.dae
- added link 5:wheel; visual mesh filename=./raw_data/part_dae/5.dae
- added link 6:caster; visual mesh filename=./raw_data/part_dae/6.dae
- added link 7:wheel; visual mesh filename=./raw_data/part_dae/7.dae
- added link 8:caster; visual mesh filename=./raw_data/part_dae/8.dae
- added link 9:wheel; visual mesh filename=./raw_data/part_dae/9.dae
Joints:
- removed joint arm14_back16
- removed joint arm15_back16
- removed joint base11_wheel5
- removed joint caster10_base11
- removed joint caster10_wheel9_rotation
- removed joint caster2_base11
- removed joint caster2_wheel1_rotation
- removed joint caster4_base11
- removed joint caster4_wheel3_rotation
- removed joint caster6_base11
- removed joint caster6_wheel5_rotation
- removed joint caster8_base11
- removed joint caster8_wheel7_rotation
- removed joint gas lift piece12_base11
- removed joint gas lift piece12_gas lift piece13_prismatic
- removed joint gas lift piece13_seat17_rotation
- removed joint seat17_arm14
- removed joint seat17_arm15
- removed joint seat17_back16
- added joint 10:caster::11:base: type fixed, parent 10:caster, child 11:base, origin xyz=0.0 0.0 0.0 rpy=0 0 0
- added joint 10:caster::9:wheel_rotation: type revolute, parent 10:caster, child 9:wheel, origin xyz=0.00319099985063076 -9.658934985168344e-09 -0.441940002143383 rpy=0 0 0, axis 1.0 0.0 0.0, limit lower=-3.141592653589793 upper=3.141592653589793 effort=10 velocity=3
- added joint 11:base::5:wheel: type fixed, parent 11:base, child 5:wheel, origin xyz=-0.26165415346622467 -1.8829651171614614e-09 -0.086154505610466 rpy=0 0 0
- added joint 12:gas lift piece::11:base: type fixed, parent 12:gas lift piece, child 11:base, origin xyz=0.0 0.0 0.0 rpy=0 0 0
- added joint 12:gas lift piece::13:gas lift piece_translation: type prismatic, parent 12:gas lift piece, child 13:gas lift piece, origin xyz=-0.06868569145071565 0.26775474017025536 -0.22430335969031795 rpy=0 0 0, axis 0.0 1.0 0.0, limit lower=-0.0365284856855869 upper=0.00347151431441307 effort=10 velocity=3
- added joint 13:gas lift piece::17:seat_rotation: type revolute, parent 13:gas lift piece, child 17:seat, origin xyz=0.06868569145071565 0.15000275606749947 0.22220634907783016 rpy=0 0 0, axis 0.0 1.0 0.0, limit lower=-3.141592653589793 upper=3.141592653589793 effort=10 velocity=3
- added joint 14:arm::16:back: type fixed, parent 14:arm, child 16:back, origin xyz=0.0 0.0 0.0 rpy=0 0 0
- added joint 15:arm::16:back: type fixed, parent 15:arm, child 16:back, origin xyz=0.0 0.0 0.0 rpy=0 0 0
- added joint 17:seat::14:arm: type fixed, parent 17:seat, child 14:arm, origin xyz=0.0 -0.4177574962377548 0.002097010612487793 rpy=0 0 0
- added joint 17:seat::15:arm: type fixed, parent 17:seat, child 15:arm, origin xyz=0.0 -0.4177574962377548 0.002097010612487793 rpy=0 0 0
- added joint 17:seat::16:back: type fixed, parent 17:seat, child 16:back, origin xyz=0.0 -0.4177574962377548 0.002097010612487793 rpy=0 0 0
- added joint 2:caster::11:base: type fixed, parent 2:caster, child 11:base, origin xyz=0.0 0.0 0.0 rpy=0 0 0
- added joint 2:caster::1:wheel_rotation: type revolute, parent 2:caster, child 1:wheel, origin xyz=0.16592684388160706 -4.846891027421307e-09 -0.22176782367751002 rpy=0 0 0, axis 1.0 0.0 0.0, limit lower=-3.141592653589793 upper=3.141592653589793 effort=10 velocity=3
- added joint 4:caster::11:base: type fixed, parent 4:caster, child 11:base, origin xyz=0.0 0.0 0.0 rpy=0 0 0
- added joint 4:caster::3:wheel_rotation: type revolute, parent 4:caster, child 3:wheel, origin xyz=0.06868565082550049 -0.39346974258781975 0.2537205144762993 rpy=0 0 0, axis 1.0 0.0 0.0, limit lower=-3.141592653589793 upper=3.141592653589793 effort=10 velocity=3
- added joint 6:caster::11:base: type fixed, parent 6:caster, child 11:base, origin xyz=0.0 0.0 0.0 rpy=0 0 0
- added joint 6:caster::5:wheel_rotation: type revolute, parent 6:caster, child 5:wheel, origin xyz=-0.26165415346622467 -1.8829651171614614e-09 -0.086154505610466 rpy=0 0 0, axis 1.0 0.0 0.0, limit lower=-3.141592653589793 upper=3.141592653589793 effort=10 velocity=3
- added joint 8:caster::11:base: type fixed, parent 8:caster, child 11:base, origin xyz=0.0 0.0 0.0 rpy=0 0 0
- added joint 8:caster::7:wheel_rotation: type revolute, parent 8:caster, child 7:wheel, origin xyz=-0.26165415346622467 -7.880555097372621e-09 -0.3605721518397331 rpy=0 0 0, axis 1.0 0.0 0.0, limit lower=-3.141592653589793 upper=3.141592653589793 effort=10 velocity=3

Commit message: fix parent bug

File: 106.URDF (robot description, URDF)
Before this commit: robot 106, 17 links, 19 joints
Links:
- link 10:caster: geometry visual mesh filename=raw_data/part_dae/10.dae
- link 11:base: geometry visual mesh filename=raw_data/part_dae/11.dae
- link 12:gas lift piece: geometry visual mesh filename=raw_data/part_dae/12.dae
- link 13:gas lift piece: geometry visual mesh filename=raw_data/part_dae/13.dae
- link 14:arm: geometry visual mesh filename=raw_data/part_dae/14.dae
- link 15:arm: geometry visual mesh filename=raw_data/part_dae/15.dae
- link 16:back: geometry visual mesh filename=raw_data/part_dae/16.dae
- link 17:seat: geometry visual mesh filename=raw_data/part_dae/17.dae
- link 1:wheel: geometry visual mesh filename=raw_data/part_dae/1.dae
- link 2:caster: geometry visual mesh filename=raw_data/part_dae/2.dae
- link 3:wheel: geometry visual mesh filename=raw_data/part_dae/3.dae
- link 4:caster: geometry visual mesh filename=raw_data/part_dae/4.dae
- link 5:wheel: geometry visual mesh filename=raw_data/part_dae/5.dae
- link 6:caster: geometry visual mesh filename=raw_data/part_dae/6.dae
- link 7:wheel: geometry visual mesh filename=raw_data/part_dae/7.dae
- link 8:caster: geometry visual mesh filename=raw_data/part_dae/8.dae
- link 9:wheel: geometry visual mesh filename=raw_data/part_dae/9.dae

Commit message: find some bugs based on 397

File: 106.URDF (robot description, URDF)
Before this commit: robot 106, 17 links, 19 joints
Joints:
- removed joint 12:gas lift piece::13:gas lift piece_translation
- added joint 13:gas lift piece::12:gas lift piece_rotation: type revolute, parent 13:gas lift piece, child 12:gas lift piece, origin xyz=0.0197197639331532 -0.06757599860429764 0.0047402818872869165 rpy=0 0 0, axis 0.0 1.0 0.0, limit lower=-3.141592653589793 upper=3.141592653589793 effort=10 velocity=3
- joint 10:caster::9:wheel_rotation: axis 1.0 0.0 0.0 -> -1.0 0.0 0.0; origin xyz=0.00319099985063076 -9.658934985168344e-09 -0.441940002143383 rpy=0 0 0 -> xyz=0.07187665067613125 0.024287743991000088 -0.19031649827957153 rpy=0 0 0
- joint 11:base::5:wheel: origin xyz=-0.26165415346622467 -1.8829651171614614e-09 -0.086154505610466 rpy=0 0 0 -> xyz=-0.19296850264072418 0.024287751766969956 0.1654689982533455 rpy=0 0 0
- joint 12:gas lift piece::11:base: origin xyz=0.0 0.0 0.0 rpy=0 0 0 -> xyz=-2.5680730458832457e-09 -0.11304300278425217 -0.028758065351089032 rpy=0 0 0
- joint 13:gas lift piece::17:seat_rotation: origin xyz=0.06868569145071565 0.15000275606749947 0.22220634907783016 rpy=0 0 0 -> xyz=0.007225165630961563 0.22200000000000003 -0.0008312173409099934 rpy=0 0 0
- joint 17:seat::14:arm: origin xyz=0.0 -0.4177574962377548 0.002097010612487793 rpy=0 0 0 -> xyz=0.01249459573411859 -0.40261900138854984 -0.023186566122892122 rpy=0 0 0
- joint 17:seat::15:arm: origin xyz=0.0 -0.4177574962377548 0.002097010612487793 rpy=0 0 0 -> xyz=0.01249459573411859 -0.40261900138854984 -0.023186566122892122 rpy=0 0 0
- joint 17:seat::16:back: origin xyz=0.0 -0.4177574962377548 0.002097010612487793 rpy=0 0 0 -> xyz=0.01249459573411859 -0.40261900138854984 -0.023186566122892122 rpy=0 0 0
- joint 2:caster::1:wheel_rotation: axis 1.0 0.0 0.0 -> 0.0 0.0 1.0; origin xyz=0.16592684388160706 -4.846891027421307e-09 -0.22176782367751002 rpy=0 0 0 -> xyz=0.23461249470710754 0.024287748803044046 0.02985568018630147 rpy=0 0 0
- joint 4:caster::3:wheel_rotation: axis 1.0 0.0 0.0 -> -1.0 0.0 0.0; origin xyz=0.06868565082550049 -0.39346974258781975 0.2537205144762993 rpy=0 0 0 -> xyz=0.06868565082550049 0.024287753649935073 0.2516235038638115 rpy=0 0 0
- joint 6:caster::5:wheel_rotation: axis 1.0 0.0 0.0 -> 0.0 0.0 1.0; origin xyz=-0.26165415346622467 -1.8829651171614614e-09 -0.086154505610466 rpy=0 0 0 -> xyz=-0.19296850264072418 0.024287751766969956 0.1654689982533455 rpy=0 0 0
- joint 8:caster::7:wheel_rotation: axis 1.0 0.0 0.0 -> 0.0 0.0 1.0; origin xyz=-0.26165415346622467 -7.880555097372621e-09 -0.3605721518397331 rpy=0 0 0 -> xyz=-0.19296850264072418 0.024287745769379976 -0.10894864797592163 rpy=0 0 0
