Commit message: update based on condensed data

File: 397.URDF (robot description, URDF)
Before this commit: robot 397, 14 links, 19 joints
Links:
- removed link 10:side panel
- removed link 11:drawer
- removed link 12:drawer
- removed link 13:drawer
- removed link 14:drawer
- removed link 1:handle
- removed link 2:handle
- removed link 3:handle
- removed link 4:handle
- removed link 5:bottom panel
- removed link 6:front panel
- removed link 7:top panel
- removed link 8:side panel
- removed link 9:back panel
- added link 0:virtual; visual cylinder length=0 radius=0
- added link 1:static; visual mesh filename=raw_data/397/part_meshes/1.dae
- added link 2:drawer 1; visual mesh filename=raw_data/397/part_meshes/2.dae
- added link 3:drawer 2; visual mesh filename=raw_data/397/part_meshes/3.dae
- added link 4:drawer 3; visual mesh filename=raw_data/397/part_meshes/4.dae
- added link 5:drawer 4; visual mesh filename=raw_data/397/part_meshes/5.dae
Joints:
- removed joint 10:side panel::5:bottom panel
- removed joint 10:side panel::6:front panel
- removed joint 10:side panel::9:back panel
- removed joint 11:drawer::4:handle
- removed joint 12:drawer::1:handle
- removed joint 13:drawer::2:handle
- removed joint 14:drawer::3:handle
- removed joint 5:bottom panel::6:front panel
- removed joint 5:bottom panel::9:back panel
- removed joint 7:top panel::10:side panel
- removed joint 7:top panel::8:side panel
- removed joint 7:top panel::9:back panel
- removed joint 8:side panel::11:drawer_translation
- removed joint 8:side panel::12:drawer_translation
- removed joint 8:side panel::13:drawer_translation
- removed joint 8:side panel::14:drawer_translation
- removed joint 8:side panel::5:bottom panel
- removed joint 8:side panel::6:front panel
- removed joint 8:side panel::9:back panel
- added joint 0:virtual::1:static: type fixed, parent 0:virtual, child 1:static, origin xyz=0.0 0.0 0.0 rpy=0 0 0
- added joint 0:virtual::2:drawer 1_translation: type prismatic, parent 0:virtual, child 2:drawer 1, origin xyz=-5.4001808166503906e-05 0.7689925134181976 -0.002888500690460205 rpy=0 0 0, axis 0.0 0.0 1.0, limit lower=-0.0001615035533905 upper=0.32883849644661 effort=10 velocity=3
- added joint 0:virtual::3:drawer 2_translation: type prismatic, parent 0:virtual, child 3:drawer 2, origin xyz=-5.4001808166503906e-05 0.57362499833107 -0.002888500690460205 rpy=0 0 0, axis 0.0 0.0 1.0, limit lower=-0.0001615035533905 upper=0.32883849644661 effort=10 velocity=3
- added joint 0:virtual::4:drawer 3_translation: type prismatic, parent 0:virtual, child 4:drawer 3, origin xyz=-5.4001808166503906e-05 0.3823090046644211 -0.002888500690460205 rpy=0 0 0, axis 0.0 0.0 1.0, limit lower=-0.0001615035533905 upper=0.32883849644661 effort=10 velocity=3
- added joint 0:virtual::5:drawer 4_translation: type prismatic, parent 0:virtual, child 5:drawer 4, origin xyz=-5.4001808166503906e-05 0.18896714970469475 -0.002888500690460205 rpy=0 0 0, axis 0.0 0.0 1.0, limit lower=-0.0001615035533905 upper=0.32883849644661 effort=10 velocity=3

File: perfect.URDF (robot description, URDF)
Before this commit: robot 397, 14 links, 19 joints
Links:
- link 1:handle: geometry visual cylinder length=0 radius=0.03
