Commit message: adjust the URDF structure

File: URDF/101.URDF (robot description, URDF)
Before this commit: robot 101, 5 links, 4 joints
Links:
- link 1:static: geometry visual mesh filename=../raw_data/101/part_meshes/1.dae
- link 2:dial 1: geometry visual mesh filename=../raw_data/101/part_meshes/2.dae
- link 3:dial 2: geometry visual mesh filename=../raw_data/101/part_meshes/3.dae
- link 4:oven door 1: geometry visual mesh filename=../raw_data/101/part_meshes/4.dae

File: URDF/106.URDF (robot description, URDF)
Before this commit: robot 106, 14 links, 13 joints
Links:
- link 10:caster 2: geometry visual mesh filename=../raw_data/106/part_meshes/10.dae
- link 11:caster 3: geometry visual mesh filename=../raw_data/106/part_meshes/11.dae
- link 12:caster 4: geometry visual mesh filename=../raw_data/106/part_meshes/12.dae
- link 13:caster 5: geometry visual mesh filename=../raw_data/106/part_meshes/13.dae
- link 1:back 1: geometry visual mesh filename=../raw_data/106/part_meshes/1.dae
- link 2:seat 1: geometry visual mesh filename=../raw_data/106/part_meshes/2.dae
- link 3:wheel 1: geometry visual mesh filename=../raw_data/106/part_meshes/3.dae
- link 4:wheel 2: geometry visual mesh filename=../raw_data/106/part_meshes/4.dae
- link 5:wheel 3: geometry visual mesh filename=../raw_data/106/part_meshes/5.dae
- link 6:wheel 4: geometry visual mesh filename=../raw_data/106/part_meshes/6.dae
- link 7:wheel 5: geometry visual mesh filename=../raw_data/106/part_meshes/7.dae
- link 8:gas lift piece 1: geometry visual mesh filename=../raw_data/106/part_meshes/8.dae
- link 9:caster 1: geometry visual mesh filename=../raw_data/106/part_meshes/9.dae

File: URDF/107.URDF (robot description, URDF)
Before this commit: robot 107, 5 links, 4 joints
Links:
- link 1:static: geometry visual mesh filename=../raw_data/107/part_meshes/1.dae
- link 2:drawer 1: geometry visual mesh filename=../raw_data/107/part_meshes/2.dae
- link 3:drawer 2: geometry visual mesh filename=../raw_data/107/part_meshes/3.dae
- link 4:cabinet door 1: geometry visual mesh filename=../raw_data/107/part_meshes/4.dae

File: URDF/108.URDF (robot description, URDF)
Before this commit: robot 108, 3 links, 2 joints
Links:
- link 1:static: geometry visual mesh filename=../raw_data/108/part_meshes/1.dae
- link 2:cabinet door 1: geometry visual mesh filename=../raw_data/108/part_meshes/2.dae

File: URDF/122.URDF (robot description, URDF)
Before this commit: robot 122, 4 links, 3 joints
Links:
- link 1:static: geometry visual mesh filename=../raw_data/122/part_meshes/1.dae
- link 2:door 1: geometry visual mesh filename=../raw_data/122/part_meshes/2.dae
- link 3:handle 2: geometry visual mesh filename=../raw_data/122/part_meshes/3.dae

File: URDF/125.URDF (robot description, URDF)
Before this commit: robot 125, 6 links, 5 joints
Links:
- link 1:static: geometry visual mesh filename=../raw_data/125/part_meshes/1.dae
- link 2:cabinet door 1: geometry visual mesh filename=../raw_data/125/part_meshes/2.dae
- link 3:cabinet door 2: geometry visual mesh filename=../raw_data/125/part_meshes/3.dae
- link 4:faucet handle 1: geometry visual mesh filename=../raw_data/125/part_meshes/4.dae
- link 5:faucet spout 1: geometry visual mesh filename=../raw_data/125/part_meshes/5.dae

File: URDF/129.URDF (robot description, URDF)
Before this commit: robot 129, 8 links, 7 joints
Links:
- link 1:static: geometry visual mesh filename=../raw_data/129/part_meshes/1.dae
- link 2:drawer 1: geometry visual mesh filename=../raw_data/129/part_meshes/2.dae
- link 3:drawer 2: geometry visual mesh filename=../raw_data/129/part_meshes/3.dae
- link 4:drawer 3: geometry visual mesh filename=../raw_data/129/part_meshes/4.dae
- link 5:drawer 4: geometry visual mesh filename=../raw_data/129/part_meshes/5.dae
- link 6:cabinet door 1: geometry visual mesh filename=../raw_data/129/part_meshes/6.dae
- link 7:drawer 5: geometry visual mesh filename=../raw_data/129/part_meshes/7.dae

File: URDF/132.URDF (robot description, URDF)
Before this commit: robot 132, 4 links, 3 joints
Links:
- link 1:static: geometry visual mesh filename=../raw_data/132/part_meshes/1.dae
- link 2:faucet handle 1: geometry visual mesh filename=../raw_data/132/part_meshes/2.dae
- link 3:faucet handle 2: geometry visual mesh filename=../raw_data/132/part_meshes/3.dae

File: URDF/133.URDF (robot description, URDF)
Before this commit: robot 133, 5 links, 4 joints
Links:
- link 1:static: geometry visual mesh filename=../raw_data/133/part_meshes/1.dae
- link 2:door 1: geometry visual mesh filename=../raw_data/133/part_meshes/2.dae
- link 3:door 2: geometry visual mesh filename=../raw_data/133/part_meshes/3.dae
- link 4:handle 1: geometry visual mesh filename=../raw_data/133/part_meshes/4.dae

File: URDF/140.URDF (robot description, URDF)
Before this commit: robot 140, 5 links, 4 joints
Links:
- link 1:static: geometry visual mesh filename=../raw_data/140/part_meshes/1.dae
- link 2:drawer 1: geometry visual mesh filename=../raw_data/140/part_meshes/2.dae
- link 3:drawer 2: geometry visual mesh filename=../raw_data/140/part_meshes/3.dae
- link 4:drawer 3: geometry visual mesh filename=../raw_data/140/part_meshes/4.dae

File: URDF/181.URDF (robot description, URDF)
Before this commit: robot 181, 4 links, 3 joints
Links:
- link 1:static: geometry visual mesh filename=../raw_data/181/part_meshes/1.dae
- link 2:cabinet door 1: geometry visual mesh filename=../raw_data/181/part_meshes/2.dae
- link 3:cabinet door 2: geometry visual mesh filename=../raw_data/181/part_meshes/3.dae

File: URDF/182.URDF (robot description, URDF)
Before this commit: robot 182, 4 links, 3 joints
Links:
- link 1:static: geometry visual mesh filename=../raw_data/182/part_meshes/1.dae
- link 2:cabinet door 1: geometry visual mesh filename=../raw_data/182/part_meshes/2.dae
- link 3:cabinet door 2: geometry visual mesh filename=../raw_data/182/part_meshes/3.dae

File: URDF/183.URDF (robot description, URDF)
Before this commit: robot 183, 5 links, 4 joints
Links:
- link 1:static: geometry visual mesh filename=../raw_data/183/part_meshes/1.dae
- link 2:drawer 1: geometry visual mesh filename=../raw_data/183/part_meshes/2.dae
- link 3:faucet handle 1: geometry visual mesh filename=../raw_data/183/part_meshes/3.dae
- link 4:faucet handle 2: geometry visual mesh filename=../raw_data/183/part_meshes/4.dae

File: URDF/184.URDF (robot description, URDF)
Before this commit: robot 184, 9 links, 8 joints
Links:
- link 1:static: geometry visual mesh filename=../raw_data/184/part_meshes/1.dae
- link 2:drawer 1: geometry visual mesh filename=../raw_data/184/part_meshes/2.dae
- link 3:drawer 2: geometry visual mesh filename=../raw_data/184/part_meshes/3.dae
- link 4:drawer 3: geometry visual mesh filename=../raw_data/184/part_meshes/4.dae
- link 5:drawer 4: geometry visual mesh filename=../raw_data/184/part_meshes/5.dae
- link 6:cabinet door 1: geometry visual mesh filename=../raw_data/184/part_meshes/6.dae
- link 7:cabinet door 2: geometry visual mesh filename=../raw_data/184/part_meshes/7.dae
- link 8:cabinet door 3: geometry visual mesh filename=../raw_data/184/part_meshes/8.dae

File: URDF/186.URDF (robot description, URDF)
Before this commit: robot 186, 6 links, 5 joints
Links:
- link 1:static: geometry visual mesh filename=../raw_data/186/part_meshes/1.dae
- link 2:faucet spout 1: geometry visual mesh filename=../raw_data/186/part_meshes/2.dae
- link 3:drawer 1: geometry visual mesh filename=../raw_data/186/part_meshes/3.dae
- link 4:drawer 2: geometry visual mesh filename=../raw_data/186/part_meshes/4.dae
- link 5:faucet handle 1: geometry visual mesh filename=../raw_data/186/part_meshes/5.dae

File: URDF/187.URDF (robot description, URDF)
Before this commit: robot 187, 5 links, 4 joints
Links:
- link 1:static: geometry visual mesh filename=../raw_data/187/part_meshes/1.dae
- link 2:door 1: geometry visual mesh filename=../raw_data/187/part_meshes/2.dae
- link 3:door 2: geometry visual mesh filename=../raw_data/187/part_meshes/3.dae
- link 4:door 3: geometry visual mesh filename=../raw_data/187/part_meshes/4.dae

File: URDF/194.URDF (robot description, URDF)
Before this commit: robot 194, 4 links, 3 joints
Links:
- link 1:static: geometry visual mesh filename=../raw_data/194/part_meshes/1.dae
- link 2:cabinet door 1: geometry visual mesh filename=../raw_data/194/part_meshes/2.dae
- link 3:cabinet door 2: geometry visual mesh filename=../raw_data/194/part_meshes/3.dae

File: URDF/214.URDF (robot description, URDF)
Before this commit: robot 214, 3 links, 2 joints
Links:
- link 1:static: geometry visual mesh filename=../raw_data/214/part_meshes/1.dae
- link 2:door 1: geometry visual mesh filename=../raw_data/214/part_meshes/2.dae

File: URDF/246.URDF (robot description, URDF)
Before this commit: robot 246, 3 links, 2 joints
Links:
- link 1:static: geometry visual mesh filename=../raw_data/246/part_meshes/1.dae
- link 2:door 1: geometry visual mesh filename=../raw_data/246/part_meshes/2.dae

File: URDF/247.URDF (robot description, URDF)
Before this commit: robot 247, 3 links, 2 joints
Links:
- link 1:static: geometry visual mesh filename=../raw_data/247/part_meshes/1.dae
- link 2:door 1: geometry visual mesh filename=../raw_data/247/part_meshes/2.dae
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
Commit message: update URDF models

File: URDF/101.URDF (robot description, URDF)
Before this commit: robot 101, 5 links, 4 joints
Links:
- link 1:static: mass None -> 1.0
- link 2:dial 1: mass None -> 1.0
- link 3:dial 2: mass None -> 1.0
- link 4:oven door 1: mass None -> 1.0

File: URDF/106.URDF (robot description, URDF)
Before this commit: robot 106, 14 links, 13 joints
Links:
- link 10:caster 2: mass None -> 1.0
- link 11:caster 3: mass None -> 1.0
- link 12:caster 4: mass None -> 1.0
- link 13:caster 5: mass None -> 1.0
- link 1:back 1: mass None -> 1.0
- link 2:seat 1: mass None -> 1.0
- link 3:wheel 1: mass None -> 1.0
- link 4:wheel 2: mass None -> 1.0
- link 5:wheel 3: mass None -> 1.0
- link 6:wheel 4: mass None -> 1.0
- link 7:wheel 5: mass None -> 1.0
- link 8:gas lift piece 1: mass None -> 1.0
- link 9:caster 1: mass None -> 1.0

File: URDF/107.URDF (robot description, URDF)
Before this commit: robot 107, 5 links, 4 joints
Links:
- link 1:static: mass None -> 1.0
- link 2:drawer 1: mass None -> 1.0
- link 3:drawer 2: mass None -> 1.0
- link 4:cabinet door 1: mass None -> 1.0

File: URDF/108.URDF (robot description, URDF)
Before this commit: robot 108, 3 links, 2 joints
Links:
- link 1:static: mass None -> 1.0
- link 2:cabinet door 1: mass None -> 1.0

File: URDF/122.URDF (robot description, URDF)
Before this commit: robot 122, 4 links, 3 joints
Links:
- link 1:static: mass None -> 1.0
- link 2:door 1: mass None -> 1.0
- link 3:handle 2: mass None -> 1.0

File: URDF/125.URDF (robot description, URDF)
Before this commit: robot 125, 6 links, 5 joints
Links:
- link 1:static: mass None -> 1.0
- link 2:cabinet door 1: mass None -> 1.0
- link 3:cabinet door 2: mass None -> 1.0
- link 4:faucet handle 1: mass None -> 1.0
- link 5:faucet spout 1: mass None -> 1.0

File: URDF/129.URDF (robot description, URDF)
Before this commit: robot 129, 8 links, 7 joints
Links:
- link 1:static: mass None -> 1.0
- link 2:drawer 1: mass None -> 1.0
- link 3:drawer 2: mass None -> 1.0
- link 4:drawer 3: mass None -> 1.0
- link 5:drawer 4: mass None -> 1.0
- link 6:cabinet door 1: mass None -> 1.0
- link 7:drawer 5: mass None -> 1.0

File: URDF/132.URDF (robot description, URDF)
Before this commit: robot 132, 4 links, 3 joints
Links:
- link 1:static: mass None -> 1.0
- link 2:faucet handle 1: mass None -> 1.0
- link 3:faucet handle 2: mass None -> 1.0

File: URDF/133.URDF (robot description, URDF)
Before this commit: robot 133, 5 links, 4 joints
Links:
- link 1:static: mass None -> 1.0
- link 2:door 1: mass None -> 1.0
- link 3:door 2: mass None -> 1.0
- link 4:handle 1: mass None -> 1.0

File: URDF/140.URDF (robot description, URDF)
Before this commit: robot 140, 5 links, 4 joints
Links:
- link 1:static: mass None -> 1.0
- link 2:drawer 1: mass None -> 1.0
- link 3:drawer 2: mass None -> 1.0
- link 4:drawer 3: mass None -> 1.0

File: URDF/181.URDF (robot description, URDF)
Before this commit: robot 181, 4 links, 3 joints
Links:
- link 1:static: mass None -> 1.0
- link 2:cabinet door 1: mass None -> 1.0
- link 3:cabinet door 2: mass None -> 1.0

File: URDF/182.URDF (robot description, URDF)
Before this commit: robot 182, 4 links, 3 joints
Links:
- link 1:static: mass None -> 1.0
- link 2:cabinet door 1: mass None -> 1.0
- link 3:cabinet door 2: mass None -> 1.0

File: URDF/183.URDF (robot description, URDF)
Before this commit: robot 183, 5 links, 4 joints
Links:
- link 1:static: mass None -> 1.0
- link 2:drawer 1: mass None -> 1.0
- link 3:faucet handle 1: mass None -> 1.0
- link 4:faucet handle 2: mass None -> 1.0

File: URDF/184.URDF (robot description, URDF)
Before this commit: robot 184, 9 links, 8 joints
Links:
- link 1:static: mass None -> 1.0
- link 2:drawer 1: mass None -> 1.0
- link 3:drawer 2: mass None -> 1.0
- link 4:drawer 3: mass None -> 1.0
- link 5:drawer 4: mass None -> 1.0
- link 6:cabinet door 1: mass None -> 1.0
- link 7:cabinet door 2: mass None -> 1.0
- link 8:cabinet door 3: mass None -> 1.0

File: URDF/186.URDF (robot description, URDF)
Before this commit: robot 186, 6 links, 5 joints
Links:
- link 1:static: mass None -> 1.0
- link 2:faucet spout 1: mass None -> 1.0
- link 3:drawer 1: mass None -> 1.0
- link 4:drawer 2: mass None -> 1.0
- link 5:faucet handle 1: mass None -> 1.0

File: URDF/187.URDF (robot description, URDF)
Before this commit: robot 187, 5 links, 4 joints
Links:
- link 1:static: mass None -> 1.0
- link 2:door 1: mass None -> 1.0
- link 3:door 2: mass None -> 1.0
- link 4:door 3: mass None -> 1.0

File: URDF/194.URDF (robot description, URDF)
Before this commit: robot 194, 4 links, 3 joints
Links:
- link 1:static: mass None -> 1.0
- link 2:cabinet door 1: mass None -> 1.0
- link 3:cabinet door 2: mass None -> 1.0

File: URDF/214.URDF (robot description, URDF)
Before this commit: robot 214, 3 links, 2 joints
Links:
- link 1:static: mass None -> 1.0
- link 2:door 1: mass None -> 1.0

File: URDF/246.URDF (robot description, URDF)
Before this commit: robot 246, 3 links, 2 joints
Links:
- link 1:static: mass None -> 1.0
- link 2:door 1: mass None -> 1.0

File: URDF/247.URDF (robot description, URDF)
Before this commit: robot 247, 3 links, 2 joints
Links:
- link 1:static: mass None -> 1.0
- link 2:door 1: mass None -> 1.0
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